File: bus_interface.sch (KiCad schematic (older format))
At the start: 11 parts, among them J5 Conn_ISA_8bit, U11 74HCT125, U4 74ALVC164245, U5 74ALVC164245

Commit message: Fix BOM swap of 1u and 4.7u caps
Parts:
- C23, C24, C25, C26: Mouser 187-CL10A475KP8NNNC -> 810-CGA3E1X7R1C105AC
Changed lines of the file:
@@
 F 2 "Passive:CAPC1608X100" H 2350 6100 50  0001 C CNN
 F 3 "~" H 2350 6100 50  0001 C CNN
-F 4 "187-CL10A475KP8NNNC" H -1650 -1100 50  0001 C CNN "Mouser"
+F 4 "810-CGA3E1X7R1C105AC" H -1650 -1100 50  0001 C CNN "Mouser"
 	1    2350 6100
 	1    0    0    -1
@@
 F 2 "Passive:CAPC1608X100" H 2700 6100 50  0001 C CNN
 F 3 "~" H 2700 6100 50  0001 C CNN
-F 4 "187-CL10A475KP8NNNC" H -1550 -1100 50  0001 C CNN "Mouser"
+F 4 "810-CGA3E1X7R1C105AC" H -1550 -1100 50  0001 C CNN "Mouser"
 	1    2700 6100
 	1    0    0    -1
@@
 F 2 "Passive:CAPC1608X100" H 3050 6100 50  0001 C CNN
 F 3 "~" H 3050 6100 50  0001 C CNN
-F 4 "187-CL10A475KP8NNNC" H -1500 -1100 50  0001 C CNN "Mouser"
+F 4 "810-CGA3E1X7R1C105AC" H -1500 -1100 50  0001 C CNN "Mouser"
 	1    3050 6100
 	1    0    0    -1
@@
 F 2 "Passive:CAPC1608X100" H 3400 6100 50  0001 C CNN
 F 3 "~" H 3400 6100 50  0001 C CNN
-F 4 "187-CL10A475KP8NNNC" H -1400 -1100 50  0001 C CNN "Mouser"
+F 4 "810-CGA3E1X7R1C105AC" H -1400 -1100 50  0001 C CNN "Mouser"
 	1    3400 6100
 	1    0    0    -1
