File: isavideo.sch (KiCad schematic (older format))
At the start: 39 parts, among them J1 PROG, J2 DE15, J3 NTSC, J4 DE9, J6 RFMOD, SW1 SW_DIP_x04, U1 ICE40HX4K-TQ144, U11 74HCT125, U2 SST26VF080A-104I/SN, U3 74ALVC164245, X1 10MHz, X2 14.318MHz

Commit message: Fix BOM swap of 1u and 4.7u caps
Parts:
- C1, C20, C21, C22, C30, C31: Mouser 187-CL10A475KP8NNNC -> 810-CGA3E1X7R1C105AC
Changed lines of the file:
@@
 F 2 "Passive:CAPC1608X100" H 6150 2050 50  0001 C CNN
 F 3 "~" H 6150 2050 50  0001 C CNN
-F 4 "187-CL10A475KP8NNNC" H 0   0   50  0001 C CNN "Mouser"
+F 4 "810-CGA3E1X7R1C105AC" H 0   0   50  0001 C CNN "Mouser"
 	1    6150 2050
 	1    0    0    -1
@@
 F 2 "Passive:CAPC1608X100" H 10000 5950 50  0001 C CNN
 F 3 "~" H 10000 5950 50  0001 C CNN
-F 4 "187-CL10A475KP8NNNC" H -100 0   50  0001 C CNN "Mouser"
+F 4 "810-CGA3E1X7R1C105AC" H -100 0   50  0001 C CNN "Mouser"
 	1    10000 5950
 	1    0    0    -1
@@
 F 2 "Passive:CAPC1608X100" H 10350 5950 50  0001 C CNN
 F 3 "~" H 10350 5950 50  0001 C CNN
-F 4 "187-CL10A475KP8NNNC" H 0   0   50  0001 C CNN "Mouser"
+F 4 "810-CGA3E1X7R1C105AC" H 0   0   50  0001 C CNN "Mouser"
 	1    10350 5950
 	1    0    0    -1
@@
 F 2 "Passive:CAPC1608X100" H 6050 3850 50  0001 C CNN
 F 3 "~" H 6050 3850 50  0001 C CNN
-F 4 "187-CL10A475KP8NNNC" H 0   0   50  0001 C CNN "Mouser"
+F 4 "810-CGA3E1X7R1C105AC" H 0   0   50  0001 C CNN "Mouser"
 	1    6050 3850
 	1    0    0    -1
@@
 F 2 "Passive:CAPC1608X100" H 6350 5700 50  0001 C CNN
 F 3 "~" H 6350 5700 50  0001 C CNN
-F 4 "187-CL10A475KP8NNNC" H 200 3650 50  0001 C CNN "Mouser"
+F 4 "810-CGA3E1X7R1C105AC" H 200 3650 50  0001 C CNN "Mouser"
 	1    6350 5700
 	1    0    0    -1
@@
 F 2 "Passive:CAPC1608X100" H 3700 5600 50  0001 C CNN
 F 3 "~" H 3700 5600 50  0001 C CNN
-F 4 "187-CL10A475KP8NNNC" H -2450 3550 50  0001 C CNN "Mouser"
+F 4 "810-CGA3E1X7R1C105AC" H -2450 3550 50  0001 C CNN "Mouser"
 	1    3700 5600
 	1    0    0    -1
@@
 Text Notes 5900 5000 0    50   ~ 0
 STUFF R25 FOR ONBOARD 14.318MHZ\nSTUFF R11 FOR ISA BUS 14.318MHZ
-Wire Bus Line
-	2050 5300 2050 5450
-Wire Bus Line
-	7750 1200 7750 1700
-Wire Bus Line
-	4800 750  4800 1250
-Wire Bus Line
-	2000 1050 2000 3850
-Wire Bus Line
-	7750 2500 7750 3000
-Wire Bus Line
-	2050 5450 2050 6000
-Wire Bus Line
-	1900 4900 1900 5550
-Wire Bus Line
-	7750 1800 7750 2400
-Wire Bus Line
-	1900 5550 1900 7300
-Wire Bus Line
-	2100 950  2100 3050
 Text Label 4550 2050 0    50   ~ 0
 OSC10M
+Wire Bus Line
+	2050 5300 2050 5450
+Wire Bus Line
+	7750 1200 7750 1700
+Wire Bus Line
+	4800 750  4800 1250
+Wire Bus Line
+	2000 1050 2000 3850
+Wire Bus Line
+	7750 2500 7750 3000
+Wire Bus Line
+	2050 5450 2050 6000
+Wire Bus Line
+	1900 4900 1900 5550
+Wire Bus Line
+	7750 1800 7750 2400
+Wire Bus Line
+	1900 5550 1900 7300
+Wire Bus Line
+	2100 950  2100 3050
 $EndSCHEMATC
