File: power.sch (KiCad schematic (older format))
At the start: 25 parts, among them U1 ICE40HX4K-TQ144, U10 APX803S00-29SA-7, U8 AP2114HA-3.3, U9 AP2114HA-1.2

Commit message: Fix BOM swap of 1u and 4.7u caps
Parts:
- C10, C11, C13, C14, C15, C16, C17, C7, C8, C9: Mouser 187-CL10A475KP8NNNC -> 810-CGA3E1X7R1C105AC
- C12, C18, C19, C2, C3, C4, C5, C6: Mouser 810-CGA3E1X7R1C105AC -> 187-CL10A475KP8NNNC
Changed lines of the file:
@@
 F 2 "Passive:CAPC1608X100" H 1500 2000 50  0001 C CNN
 F 3 "~" H 1500 2000 50  0001 C CNN
-F 4 "810-CGA3E1X7R1C105AC" H 0   0   50  0001 C CNN "Mouser"
+F 4 "187-CL10A475KP8NNNC" H 0   0   50  0001 C CNN "Mouser"
 	1    1500 2000
 	1    0    0    -1
@@
 F 2 "Passive:CAPC1608X100" H 2450 2000 50  0001 C CNN
 F 3 "~" H 2450 2000 50  0001 C CNN
-F 4 "810-CGA3E1X7R1C105AC" H 0   0   50  0001 C CNN "Mouser"
+F 4 "187-CL10A475KP8NNNC" H 0   0   50  0001 C CNN "Mouser"
 	1    2450 2000
 	1    0    0    -1
@@
 F 2 "Passive:CAPC1608X100" H 1500 3600 50  0001 C CNN
 F 3 "~" H 1500 3600 50  0001 C CNN
-F 4 "810-CGA3E1X7R1C105AC" H 0   0   50  0001 C CNN "Mouser"
+F 4 "187-CL10A475KP8NNNC" H 0   0   50  0001 C CNN "Mouser"
 	1    1500 3600
 	1    0    0    -1
@@
 F 2 "Passive:CAPC1608X100" H 2450 3600 50  0001 C CNN
 F 3 "~" H 2450 3600 50  0001 C CNN
-F 4 "810-CGA3E1X7R1C105AC" H 0   0   50  0001 C CNN "Mouser"
+F 4 "187-CL10A475KP8NNNC" H 0   0   50  0001 C CNN "Mouser"
 	1    2450 3600
 	1    0    0    -1
@@
 F 2 "Passive:CAPC1608X100" H 6900 4950 50  0001 C CNN
 F 3 "~" H 6900 4950 50  0001 C CNN
-F 4 "810-CGA3E1X7R1C105AC" H 0   0   50  0001 C CNN "Mouser"
+F 4 "187-CL10A475KP8NNNC" H 0   0   50  0001 C CNN "Mouser"
 	1    6900 4950
 	1    0    0    -1
@@
 F 2 "Passive:CAPC1608X100" H 7550 4950 50  0001 C CNN
 F 3 "~" H 7550 4950 50  0001 C CNN
-F 4 "810-CGA3E1X7R1C105AC" H 0   0   50  0001 C CNN "Mouser"
+F 4 "187-CL10A475KP8NNNC" H 0   0   50  0001 C CNN "Mouser"
 	1    7550 4950
 	1    0    0    -1
@@
 F 2 "Passive:CAPC1608X100" H 7250 4950 50  0001 C CNN
 F 3 "~" H 7250 4950 50  0001 C CNN
-F 4 "187-CL10A475KP8NNNC" H 0   0   50  0001 C CNN "Mouser"
+F 4 "810-CGA3E1X7R1C105AC" H 0   0   50  0001 C CNN "Mouser"
 	1    7250 4950
 	1    0    0    -1
@@
 F 2 "Passive:CAPC1608X100" H 7900 4950 50  0001 C CNN
 F 3 "~" H 7900 4950 50  0001 C CNN
-F 4 "187-CL10A475KP8NNNC" H 0   0   50  0001 C CNN "Mouser"
+F 4 "810-CGA3E1X7R1C105AC" H 0   0   50  0001 C CNN "Mouser"
 	1    7900 4950
 	1    0    0    -1
@@
 F 2 "Passive:CAPC1608X100" H 7200 4250 50  0001 C CNN
 F 3 "~" H 7200 4250 50  0001 C CNN
-F 4 "187-CL10A475KP8NNNC" H 0   0   50  0001 C CNN "Mouser"
+F 4 "810-CGA3E1X7R1C105AC" H 0   0   50  0001 C CNN "Mouser"
 	1    7200 4250
 	1    0    0    -1
@@
 F 2 "Passive:CAPC1608X100" H 7450 4250 50  0001 C CNN
 F 3 "~" H 7450 4250 50  0001 C CNN
-F 4 "187-CL10A475KP8NNNC" H 0   0   50  0001 C CNN "Mouser"
+F 4 "810-CGA3E1X7R1C105AC" H 0   0   50  0001 C CNN "Mouser"
 	1    7450 4250
 	1    0    0    -1
@@
 F 2 "Passive:CAPC1608X100" H 7700 4250 50  0001 C CNN
 F 3 "~" H 7700 4250 50  0001 C CNN
-F 4 "187-CL10A475KP8NNNC" H 0   0   50  0001 C CNN "Mouser"
+F 4 "810-CGA3E1X7R1C105AC" H 0   0   50  0001 C CNN "Mouser"
 	1    7700 4250
 	1    0    0    -1
@@
 F 2 "Passive:CAPC1608X100" H 7950 4250 50  0001 C CNN
 F 3 "~" H 7950 4250 50  0001 C CNN
-F 4 "187-CL10A475KP8NNNC" H 0   0   50  0001 C CNN "Mouser"
+F 4 "810-CGA3E1X7R1C105AC" H 0   0   50  0001 C CNN "Mouser"
 	1    7950 4250
 	1    0    0    -1
@@
 F 2 "Passive:CAPC1608X100" H 8200 4250 50  0001 C CNN
 F 3 "~" H 8200 4250 50  0001 C CNN
-F 4 "810-CGA3E1X7R1C105AC" H 0   0   50  0001 C CNN "Mouser"
+F 4 "187-CL10A475KP8NNNC" H 0   0   50  0001 C CNN "Mouser"
 	1    8200 4250
 	1    0    0    -1
@@
 F 2 "Passive:CAPC1608X100" H 7200 3000 50  0001 C CNN
 F 3 "~" H 7200 3000 50  0001 C CNN
-F 4 "187-CL10A475KP8NNNC" H 0   0   50  0001 C CNN "Mouser"
+F 4 "810-CGA3E1X7R1C105AC" H 0   0   50  0001 C CNN "Mouser"
 	1    7200 3000
 	1    0    0    -1
@@
 F 2 "Passive:CAPC1608X100" H 7450 3000 50  0001 C CNN
 F 3 "~" H 7450 3000 50  0001 C CNN
-F 4 "187-CL10A475KP8NNNC" H 0   0   50  0001 C CNN "Mouser"
+F 4 "810-CGA3E1X7R1C105AC" H 0   0   50  0001 C CNN "Mouser"
 	1    7450 3000
 	1    0    0    -1
@@
 F 2 "Passive:CAPC1608X100" H 7700 3000 50  0001 C CNN
 F 3 "~" H 7700 3000 50  0001 C CNN
-F 4 "187-CL10A475KP8NNNC" H 0   0   50  0001 C CNN "Mouser"
+F 4 "810-CGA3E1X7R1C105AC" H 0   0   50  0001 C CNN "Mouser"
 	1    7700 3000
 	1    0    0    -1
@@
 F 2 "Passive:CAPC1608X100" H 7950 3000 50  0001 C CNN
 F 3 "~" H 7950 3000 50  0001 C CNN
-F 4 "187-CL10A475KP8NNNC" H 0   0   50  0001 C CNN "Mouser"
+F 4 "810-CGA3E1X7R1C105AC" H 0   0   50  0001 C CNN "Mouser"
 	1    7950 3000
 	1    0    0    -1
@@
 F 2 "Passive:CAPC1608X100" H 8200 3000 50  0001 C CNN
 F 3 "~" H 8200 3000 50  0001 C CNN
-F 4 "810-CGA3E1X7R1C105AC" H 0   0   50  0001 C CNN "Mouser"
+F 4 "187-CL10A475KP8NNNC" H 0   0   50  0001 C CNN "Mouser"
 	1    8200 3000
 	1    0    0    -1
