File: vga_dac.sch (KiCad schematic (older format))
At the start: 20 parts, among them U6 ADA4891-3

Commit message: Fix BOM swap of 1u and 4.7u caps
Parts:
- C27: Mouser 187-CL10A475KP8NNNC -> 810-CGA3E1X7R1C105AC
Changed lines of the file:
@@
 F 2 "Passive:CAPC1608X100" H 7100 5100 50  0001 C CNN
 F 3 "~" H 7100 5100 50  0001 C CNN
-F 4 "187-CL10A475KP8NNNC" H 0   0   50  0001 C CNN "Mouser"
+F 4 "810-CGA3E1X7R1C105AC" H 0   0   50  0001 C CNN "Mouser"
 	1    7100 5100
 	1    0    0    -1
