File: isa-video/isavideo.sch (KiCad schematic (older format))
At the start: 39 parts, among them J1 PROG, J2 DE15, J3 NTSC, J4 DE9, J6 RFMOD, SW1 SW_DIP_x04, U1 ICE40HX4K-TQ144, U11 74HCT125, U2 SST26VF080A-104I/SN, U3 74ALVC164245, X1 10MHz, X2 14.318MHz

Commit message: My Graphics gremlin hdmi
Parts:
- removed J2: DE15, Conn:DB15HDFC, symbol Connector_Generic_Shielded:Conn_01x15_Shielded
- removed J3: NTSC, Conn:KOBICONN_161-03X0-E, symbol Connector:Conn_Coaxial
- removed J4: DE9, Conn:DB9FC2, symbol Connector_Generic_Shielded:Conn_01x09_Shielded
- removed R12: 100, Passive:RESC1608X55, symbol Device:R_Small_US
- added J2: DB15_Female_HighDensity_MountingHoles, Connector_Dsub:DSUB-15-HD_Female_Horizontal_P2.29x1.98mm_EdgePinOffset8.35mm_Housed_MountingHolesOffset10.89mm, symbol Connector:DB15_Female_HighDensity_MountingHoles
- added J3: PJRAN1X1U04X, libraries:SWITCHCRAFT_PJRAN1X1U04X, symbol PJRAN1X1U04X:PJRAN1X1U04X
- C1, C20, C21, C22, C30, C31: footprint Passive:CAPC1608X100 -> Capacitor_SMD:C_0603_1608Metric
- F1: footprint Passive:RESC3216X70 -> Resistor_SMD:R_1206_3216Metric
- J1: footprint Pin_Headers:Pin_Header_Straight_2x04_Pitch2.54mm -> Connector_PinHeader_2.54mm:PinHeader_2x04_P2.54mm_Vertical
- J6: footprint Pin_Headers:Pin_Header_Straight_1x04_Pitch2.54mm -> Connector_PinHeader_2.54mm:PinHeader_1x04_P2.54mm_Vertical
- R11: Mouser DNI -> (none)
- U1: symbol logic:ICE40HX4K-TQ144 -> isavideo-rescue:ICE40HX4K-TQ144-logic
- U3: symbol logic:74ALVC164245 -> isavideo-rescue:74ALVC164245-logic
Connections:
- net labels added: HDMI_BLU, HDMI_CLK, HDMI_DE, HDMI_GRN, HDMI_HS, HDMI_INT, HDMI_PD, HDMI_RED, HDMI_VS
- net labels removed: BLUE, BLUE2, BLUE2_5V, BLUE_5V, GREEN, GREEN2, GREEN2_5V, GREEN_5V, HSYNC, HSYNC_5V, ID0, ID1_SDA, ID2, ID3_SCL, RED, RED2, RED2_5V, RED_5V, VID_EN, VSYNC, VSYNC_5V
- wire segments 352 -> 330
- no-connect marks 4 -> 25
Other:
- note added: "DESIGN BY @TubeTimeUS\nModified by @yeokm1"
- note added: "GRAPHICS GREMLIN (with HDMI)"
- note removed: "DESIGN BY @TubeTimeUS"
- note removed: "GND"
- note removed: "GRAPHICS GREMLIN"
- note removed: "INTENSITY"
- note removed: "VIDEO"
- moved on the sheet: F1, U11A, U11B
