File: isa-video/power.sch (KiCad schematic (older format))
At the start: 25 parts, among them U1 ICE40HX4K-TQ144, U10 APX803S00-29SA-7, U8 AP2114HA-3.3, U9 AP2114HA-1.2

Commit message: My Graphics gremlin hdmi
Parts:
- removed U8: AP2114HA-3.3, Active:SOT230P700X170-3, symbol Regulator_Linear:TC1262-33
- added D1, D2: Yellow, LED_SMD:LED_0603_1608Metric_Pad1.05x0.95mm_HandSolder, symbol Device:LED
- added J7: Conn_01x05, Connector_PinHeader_2.54mm:PinHeader_1x05_P2.54mm_Vertical, symbol Connector_Generic:Conn_01x05
- added R12: 2200, Resistor_SMD:R_0603_1608Metric_Pad0.98x0.95mm_HandSolder, symbol Device:R_Small_US
- added R32: 1200, Resistor_SMD:R_0603_1608Metric, symbol Device:R_Small_US
- added U8: LD1085D2T33R, Package_TO_SOT_SMD:TO-263-2, symbol Regulator_Linear:LD1086D2T33TR
- C10, C11, C12, C13, C14, C15, C16, C17, C18, C19, C3, C5, C6, C7, C8, C9: footprint Passive:CAPC1608X100 -> Capacitor_SMD:C_0603_1608Metric
- C2, C4: value 4.7u -> 10uF 16V; footprint Passive:CAPC1608X100 -> Capacitor_SMD:C_0603_1608Metric_Pad1.08x0.95mm_HandSolder; Mouser 187-CL10A475KP8NNNC -> 81-ZRB18AR61C106ME1L
- U1: symbol logic:ICE40HX4K-TQ144 -> isavideo-rescue:ICE40HX4K-TQ144-logic
Connections:
- net labels added: +12V
- wire segments 140 -> 152
Other:
- note added: "DESIGN BY @TubeTimeUS\nModified by @yeokm1"
- note added: "GRAPHICS GREMLIN (with HDMI)"
- note removed: "DESIGN BY @TubeTimeUS"
- note removed: "GRAPHICS GREMLIN"
