File: isa-video/vga_dac.sch (KiCad schematic (older format))
At the start: 20 parts, among them U6 ADA4891-3

Commit message: My Graphics gremlin hdmi
Parts:
- C27: footprint Passive:CAPC1608X100 -> Capacitor_SMD:C_0603_1608Metric
Other:
- note added: "DESIGN BY @TubeTimeUS\nModified by @yeokm1"
- note added: "GRAPHICS GREMLIN (with HDMI)"
- note removed: "DESIGN BY @TubeTimeUS"
- note removed: "GRAPHICS GREMLIN"
Changed lines of the file:
@@
 EESchema Schematic File Version 4
-LIBS:isavideo-cache
-EELAYER 29 0
+EELAYER 30 0
 EELAYER END
 $Descr A4 11693 8268
 encoding utf-8
-Sheet 3 5
+Sheet 3 6
 Title "Resistor Ladder DAC and Output Buffer"
-Date ""
-Rev "2"
+Date "2021-08-09"
+Rev "2.1"
 Comp ""
 Comment1 ""
@@
 F 0 "C27" H 7192 5146 50  0000 L CNN
 F 1 "1u" H 7192 5055 50  0000 L CNN
-F 2 "Passive:CAPC1608X100" H 7100 5100 50  0001 C CNN
+F 2 "Capacitor_SMD:C_0603_1608Metric" H 7100 5100 50  0001 C CNN
 F 3 "~" H 7100 5100 50  0001 C CNN
 F 4 "810-CGA3E1X7R1C105AC" H 0   0   50  0001 C CNN "Mouser"
@@
 ON THE ADA4891-3\nTHESE PINS ARE ALL\n~PD~ (POWER DOWN)
 Text Notes 7100 6800 0    100  ~ 0
-GRAPHICS GREMLIN
+GRAPHICS GREMLIN (with HDMI)
 Text Notes 7100 6950 0    50   ~ 0
-DESIGN BY @TubeTimeUS
+DESIGN BY @TubeTimeUS\nModified by @yeokm1
 Text Notes 550  7700 0    50   ~ 0
 This work is licensed under the Creative Commons Attribution-ShareAlike 4.0 International License. \nTo view a copy of this license, visit http://creativecommons.org/licenses/by-sa/4.0/ or send\na letter to Creative Commons, PO Box 1866, Mountain View, CA 94042, USA.
