File: isa-video/hdmi.kicad_sch (KiCad schematic)
At the start: 40 parts, among them J4 10029449-111RLF, J8 Conn_02x06_Odd_Even, U12 TFP410PAP

Commit message: Adjust TFP410 vias
Parts:
- U12: footprint Package_QFP:HTQFP-64-1EP_10x10mm_P0.5mm_EP8x8mm_Mask4.4x4.4mm_ThermalVias -> libraries:TFP410_ThermalVias
Changed lines of the file:
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@@
       (effects (font (size 1.27 1.27)))
     )
-    (property "Footprint" "Package_QFP:HTQFP-64-1EP_10x10mm_P0.5mm_EP8x8mm_Mask4.4x4.4mm_ThermalVias" (at 241.3 151.13 0)
+    (property "Footprint" "libraries:TFP410_ThermalVias" (at 241.3 151.13 0)
       (effects (font (size 1.27 1.27)) hide)
     )
