File: isa-video/isavideo.kicad_sch (KiCad schematic)
At the start: 37 parts, among them J1 PROG, J2 DB15_Female_HighDensity_Mount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, J3 PJRAN1X1U04X, J6 RFMOD, SW1 SW_DIP_x04, U1 ICE40HX4K-TQ144, U11 74HCT125, U2 SST26VF080A-104I/SN, U3 74ALVC164245, X1 10MHz, X2 14.318MHz

Commit message: minor adjustment to VGA footprint
Parts:
- J2: footprint Connector_Dsub:DSUB-15-HD_Female_Horizontal_P2.29x1.98mm_EdgePinOffset8.35mm_Housed_MountingHolesOffset10.89mm -> libraries:23117631
Changed lines of the file:
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@@
   (title_block
     (title "Top Level")
-    (date "2023-09-17")
-    (rev "2.2")
+    (date "2023-10-13")
+    (rev "2.3")
   )
   (junction (at 148.59 43.18) (diameter 0) (color 0 0 0 0)
@@
       (effects (font (size 1.27 1.27)))
     )
-    (property "Footprint" "Connector_Dsub:DSUB-15-HD_Female_Horizontal_P2.29x1.98mm_EdgePinOffset8.35mm_Housed_MountingHolesOffset10.89mm" (at 237.49 26.67 0)
+    (property "Footprint" "libraries:23117631" (at 237.49 26.67 0)
       (effects (font (size 1.27 1.27)) hide)
     )
