File: isa-video/isavideo.kicad_pcb (KiCad board)
At the start: 4 copper layers, 106.4 x 95 mm, 142 parts, among them J1 PROG, J2 DB15_Female_HighDensity_Mount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, J3 PJRAN1X1U04X, J4 10029449-111RLF, J5 Conn_ISA_8bit, J6 RFMOD, J7 Conn_01x05, J8 Conn_02x06_Odd_Even, SW1 SW_DIP_x04, U1 ICE40HX4K-TQ144, U10 APX803S00-29SA-7, U11 74HCT125, U12 TFP410PAP, U2 SST26VF080A-104I/SN, U3 74ALVC164245, U4 74ALVC164245, U5 74ALVC164245, U6 ADA4891-3, U7 IS61WV5128BLL-10KLI, U8 LD1085D2T33R, U9 AP2114HA-1.2, X1 10MHz, X2 14.318MHz

Commit message: add 3d view for VGA
Parts:
- moved J2 0.70 mm to (185.0, 56.0)
Changed lines of the file:
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@@
   )
   (footprint "libraries:23117631" locked (layer "F.Cu")
-    (at 185.7 56 90)
+    (at 185 56 90)
     (descr "2311763-1-2")
     (tags "Connector")
@@
     (pad "MH1" thru_hole circle locked (at 8.185 2.54 90) (size 4.77 4.77) (drill 3.18) (layers "*.Cu" "*.Mask"))
     (pad "MH2" thru_hole circle locked (at -16.815 2.54 90) (size 4.77 4.77) (drill 3.18) (layers "*.Cu" "*.Mask"))
+    (model "${KIPRJMOD}/libraries/c-2311763-1-b1-3d.stp"
+      (offset (xyz -4.3 -20 6.3))
+      (scale (xyz 1 1 1))
+      (rotate (xyz -90 0 0))
+    )
   )
   (footprint "Switch:SW_DIP254P762X635-8" (layer "F.Cu")
@@
     (property "ki_keywords" "r resistor")
     (attr smd)
-    (fp_text reference "R15" (at 0.78 -1.4 180) (layer "F.SilkS")
+    (fp_text reference "R15" (at 0.2 -2.35 -90) (layer "F.SilkS")
         (effects (font (size 1 1) (thickness 0.15)))
     )
@@
     (effects (font (size 1.27 1.016) (thickness 0.2032)))
   )
-  (gr_text "REGULAR OL' VGA" (at 182.1 53 90) (layer "F.SilkS")
+  (gr_text "REGULAR OL' VGA" (at 182.05 51.6 90) (layer "F.SilkS")
     (effects (font (size 1.27 1.27) (thickness 0.2032)))
   )
